File: hardware/kicad/ac.kicad_sch (KiCad schematic)
At the start: 25 parts, among them J1 AC_Input, J2 Hirose RPC1-12RB-6P(71), Q1 KIA50N06BD, Q2 KIA50N06BD, U1 VOS628A, U2 L78L24_SOT89, U3 Si8751, U4 AP2111H-3.3

Commit message: Update opensolder
Parts:
- added R21: 10k, Resistor_SMD:R_0805_2012Metric, symbol Device:R_Small
- PS1: value PDSE1-S24-S5-S -> PCSA1-S24-S5-S
Connections:
- net +3V3: now also R21.1
- net ZERO_CROSS: now also R21.2
