File: hardware/kicad/opensolder.kicad_pcb (KiCad board)
At the start: 2 copper layers, 100 x 44 mm, 69 parts, among them J1 AC_Input, J2 Hirose RPC1-12RB-6P(71), J3 SWD, J4 UART, J5 Reset_Switch, Q1 KIA50N06BD, Q2 KIA50N06BD, SW2 PEC11R-RotEnc, U1 VOS628A, U2 L78L24_SOT89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

Commit message: Update opensolder
Parts:
- added R21: 10k, Resistor_SMD:R_0805_2012Metric, F.Cu at (143.5, 93.1)
- PS1: value PDSE1-S24-S5-S -> PCSA1-S24-S5-S
- SW2: value PEC11R-RotEnc -> PEC11R-4220F-S0024
Routing:
- net +3V3: track 209.6 -> 214.5 mm
- net ZERO_CROSS: track 38.8 -> 43.3 mm
